File: PoE_Splitter.kicad_pcb (KiCad board)
At the start: 2 copper layers, 104 x 62 mm, 113 parts, among them J1 AMASS_XT30PW-M, J2 R-RJ45R10P-B000, J3 R-RJ45R10P-B000, J4 AMASS_XT30PW-M, J5 AMASS_XT30PW-M, Q1 BSS127S, U1 VCF4812EBO-120WR3-N, U2 PD70224, U3 TPS2372, U4 MPQ8875A

Commit message: 1
Parts:
- added C29: 150uF, Capacitor_SMD:CP_Elec_6.3x5.7, F.Cu at (155.4, 108.0)
- added C53: 2.2uF, Capacitor_SMD:C_1812_4532Metric, B.Cu at (186.4, 97.1)
- C26: renamed from C40; value 10uF -> 2.2uF
- C27: renamed from C41; value 10uF -> 2.2uF
- C28: renamed from C2; moved to F.Cu
- C48: renamed from C31; moved to B.Cu
- C49: renamed from C5; moved to B.Cu
- D8: renamed from D10; moved to B.Cu
- D9: moved to B.Cu
- H1, H2, H3: renamed from REF**; value MountingHole_2.2mm_M2_ISO7380 -> M2
- H4: renamed from REF**; value MountingHole_2.2mm_M2_ISO7380_Pad -> M2
- L2: footprint Inductor_SMD:L_Coilcraft_XAL8080-XXX -> Inductor_SMD:L_Chilisin_BWVS00808040
- moved C28 13.1 mm to (164.1, 107.5), turned to 0 degrees
- moved C49 12.1 mm to (176.1, 105.2), turned to 0 degrees
- moved D9 12.1 mm to (176.1, 108.3), turned to 0 degrees
- moved D10 11.6 mm to (158.9, 110.5), turned to 90 degrees
- moved C48 10.5 mm to (187.8, 105.2)
- moved D8 10.5 mm to (187.8, 108.3)
- moved J5 10.4 mm to (154.3, 115.5)
- moved FB2 10.1 mm to (109.7, 71.5)
- moved C40 10.0 mm to (182.5, 97.1)
- moved C1 10.0 mm to (121.6, 67.5)
- moved C10 10.0 mm to (103.0, 82.5)
- moved C11 10.0 mm to (109.3, 82.5)
- moved C12 10.0 mm to (103.8, 84.8)
- moved C13 10.0 mm to (108.6, 84.8)
- moved C14 10.0 mm to (157.3, 94.2)
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- renumbered C13 to C1, C28 to C10, C26 to C11, C29 to C12, C27 to C13, C33 to C14, C43 to C15, C44 to C16, C3 to C17, C3 to C18, C45 to C19, C17 to C2, C39 to C20, C34 to C21, C36 to C22, C35 to C23, C46 to C24, C42 to C25, C15 to C3, C20 to C30, C19 to C31, C1 to C32, C24 to C33, C22 to C34, C23 to C35, C30 to C36, C10 to C37, C6 to C38, C7 to C39, C16 to C4, C4 to C40, C8 to C41, C37 to C42, C9 to C43, C48 to C44, C38 to C45, C12 to C46, C11 to C47, C14 to C5, C49 to C50, C47 to C51, C21 to C6, C32 to C7, C18 to C8, C25 to C9, D7 to D1, D8 to D10, D5 to D3, D6 to D4, D1 to D5, D3 to D6, D4 to D7, FB2 to FB1, FB1 to FB2, J2 to J1, J3 to J2, J4 to J3, J5 to J4, J1 to J5, R13 to R1, R20 to R10, R19 to R11, R1 to R12, R22 to R13, R21 to R14, R14 to R15, R4 to R16, R15 to R17, R16 to R18, R2 to R19, R18 to R2, R3 to R20, R5 to R21, R12 to R22, R6 to R23, R11 to R24, R7 to R25, R10 to R26, R8 to R27, R30 to R28, R9 to R29, R25 to R3, R29 to R30, R23 to R4, R24 to R5, R28 to R6, R26 to R7, R27 to R8, R17 to R9, RV4 to RV1, RV3 to RV2, RV2 to RV3, RV1 to RV4, U3 to U2, U4 to U3, U2 to U4
Connections:
- C17 pad 1: (no net) -> VOUT+
- C17 pad 2: (no net) -> VOUT-
- C28 pad 1: VOUT+ -> PVOUT
- D10 pad 1: VOUT+ -> PVOUT
- J5 pad 2: VOUT+ -> PVOUT
- J5 pad 3: unconnected-(J1-Pin_1-Pad3) -> /SCL
- J5 pad 4: unconnected-(J1-Pin_2-Pad4) -> /SDA
- U3 pad 11: /DC-DC/SDA -> /SDA
- U3 pad 12: /DC-DC/SCL -> /SCL
Routing:
- net VOUT+: track 6.97 -> 58.9 mm, vias 0 -> 8
- net VOUT-: track 9.43 -> 60.6 mm, vias 5 -> 38
- net /SDA: track 0.00 -> 30.9 mm, vias 0 -> 1
- net /SCL: track 0.00 -> 29.4 mm, vias 0 -> 1
- net Net-(U3-EN): track 1.47 -> 7.06 mm, vias 1 -> 2
- net Net-(U3-SYNC): track 1.39 -> 5.47 mm, vias 1 -> 2
- net VDD: track 26.8 -> 30.9 mm, vias 18 -> 19
- net /DC-DC/SDA: track 1.11 -> 0.00 mm, vias 1 -> 0
- net /DC-DC/SCL: track 1.00 -> 0.00 mm, vias 1 -> 0
- net Net-(TR1-MCT3): track 2.48 -> 1.74 mm
- net /RJ45 Ports/MX4+: track 17.6 -> 16.9 mm
- net /DC-DC/PG: track 6.52 -> 5.85 mm
- net /RJ45 Ports/MX4-: track 14.7 -> 14.2 mm
- net /RJ45 Ports/MX2-: track 31.0 -> 30.4 mm
- net /RJ45 Ports/MX2+: track 33.0 -> 32.4 mm
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- added copper zone on B.Cu, net PVOUT

Commit message: add ci
Parts:
- added R31: 10kΩ, Resistor_SMD:R_0603_1608Metric, B.Cu at (159.8, 97.0)
- added R32: 10kΩ, Resistor_SMD:R_0603_1608Metric, B.Cu at (157.4, 97.8)
- added R33: 22Ω, Resistor_SMD:R_0603_1608Metric, B.Cu at (159.8, 100.0)
- added R34: 22Ω, Resistor_SMD:R_0603_1608Metric, B.Cu at (159.8, 98.5)
- added U5: USBLC6-2P6, Package_TO_SOT_SMD:SOT-666, B.Cu at (162.8, 98.1)
Connections:
- net PRE_VDD renamed VRECT+
- net PRE_VSS renamed VRECT-
- net PVOUT renamed AUX_OUT+
- U3 pad 11: /SDA -> /DC-DC/MPS_SDA
- U3 pad 12: /SCL -> /DC-DC/MPS_SCL
Routing:
- net /DC-DC/MPS_VCC: track 2.97 -> 15.1 mm
- net /SCL: track 29.4 -> 23.3 mm, vias 1 -> 0
- net /SDA: track 30.9 -> 25.7 mm, vias 1 -> 0
- net /DC-DC/MPS_SCL: track 0.00 -> 3.14 mm, vias 0 -> 1
- net /DC-DC/MPS_SDA: track 0.00 -> 2.88 mm, vias 0 -> 1
- net Net-(R33-Pad2): track 0.00 -> 1.87 mm
- net Net-(R34-Pad2): track 0.00 -> 1.69 mm
- net VOUT-: vias 38 -> 45
