File: PoE_Splitter.kicad_sch (KiCad schematic)
At the start: 18 parts, among them J1 AMASS_XT30PW-M, J4 AMASS_XT30PW-M, J5 AMASS_XT30PW-M

Commit message: 1
Parts:
- removed C2: 100nF, Capacitor_SMD:C_0805_2012Metric, symbol Device:C
- removed D8: SMAJ12A, Diode_SMD:D_SMA, symbol Diode:SMAJ12A
- removed J1: AMASS_XT30PW-M, PoE_Splitter:AMASS_XT30PW(2+2)-M_Horizontal, symbol PoE_Splitter:AMASS_XT30PW(2+2)-M
- added C28: 100nF, Capacitor_SMD:C_0805_2012Metric, symbol Device:C
- added D10: SMAJ12A, Diode_SMD:D_SMA, symbol Diode:SMAJ12A
- added H1, H2, H3: M2, MountingHole:MountingHole_2.2mm_M2_ISO7380, symbol Mechanical:MountingHole
- added H4: M2, MountingHole:MountingHole_2.2mm_M2_ISO7380_Pad, symbol Mechanical:MountingHole_Pad
- added J5: AMASS_XT30PW-M, PoE_Splitter:AMASS_XT30PW(2+2)-M_Horizontal, symbol PoE_Splitter:AMASS_XT30PW(2+2)-M
- renumbered C30 to C36, C31 to C48, C5 to C49, D7 to D1, D5 to D3, D6 to D4, D10 to D8, J4 to J3, J5 to J4, R14 to R15, R16 to R18, R25 to R3, R23 to R4, R24 to R5
Connections:
- net CHASSIS_GND: now also H4.1
- net VOUT-: now also C28.2, D10.2 (A2), J5.1 (Pin_1)
- new net DC-DC/PVOUT: C28.1, D10.1 (A1), J5.2 (Pin_2)
- new net SCL: J5.3 (Pin_1)
- new net SDA: J5.4 (Pin_2)
Other:
- sheet DC-DC ports: added PVOUT, SCL, SDA; removed none

Commit message: add ci
Connections:
- net DC-DC/PVOUT renamed AUX_OUT+
- net PRE_VSS renamed VRECT-
Other:
- sheet DC-DC ports: added none; removed PVOUT
- moved on the sheet: C28, C36, C48, C49, D1, D10, D3, D4, D8, D9, J3, J4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

Commit message: add sheet titles
Other:
- company: (none) -> Acha
- title: (none) -> PoE_Splitter
Changed lines of the file:
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@@
 	(generator_version "10.0")
 	(paper "A4")
+	(title_block
+		(title "PoE_Splitter")
+		(date "${CURRENT_DATE}")
+		(rev "${SHORT_SHA}")
+		(company "Acha")
+		(comment 1 "https://github.com/acha666/PoE_Splitter@${BRANCH}")
+		(comment 2 "GPL-3.0 Licensed")
+	)
 	(polyline
 		(pts
