File: PoE_Splitter.kicad_sch (KiCad schematic)
At the start: 22 parts, among them J3 AMASS_XT30PW-M, J4 AMASS_XT30PW-M, J5 AMASS_XT30PW-M

Commit message: minor cap footprint and value changes
Parts:
- C48, C49: footprint Capacitor_SMD:C_1808_4520Metric -> Capacitor_SMD:C_1812_4532Metric
Changed lines of the file:
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@@
 			)
 		)
-		(property "Footprint" "Capacitor_SMD:C_1808_4520Metric"
+		(property "Footprint" "Capacitor_SMD:C_1812_4532Metric"
 			(at 202.8952 101.6 0)
 			(hide yes)
@@
 			)
 		)
-		(property "Footprint" "Capacitor_SMD:C_1808_4520Metric"
+		(property "Footprint" "Capacitor_SMD:C_1812_4532Metric"
 			(at 202.8952 128.27 0)
 			(hide yes)
