File: Rectifier.kicad_sch (KiCad schematic)
At the start: 22 parts, among them U2 PD70224

Commit message: 1
Parts:
- renumbered C28 to C10, C26 to C11, C29 to C12, C27 to C13, C17 to C2, C15 to C3, C20 to C30, C19 to C31, C16 to C4, C14 to C5, C18 to C8, C25 to C9, D1 to D5, D3 to D6, FB2 to FB1, FB1 to FB2, RV4 to RV1, RV3 to RV2, RV2 to RV3, RV1 to RV4, U2 to U4
Changed lines of the file:
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@@
 		(in_pos_files yes)
 		(dnp no)
-		(property "Reference" "C15"
+		(property "Reference" "C3"
 			(at 122.174 64.516 0)
 			(show_name no)
@@
 			(project "PoE_Splitter"
 				(path "/d9db320b-7bcf-482d-be5b-dfde980903b7/135e74f4-e2a5-4ade-99ba-362d75f4aa12"
-					(reference "C15")
+					(reference "C3")
 					(unit 1)
 				)
@@
 		(in_pos_files yes)
 		(dnp no)
-		(property "Reference" "C14"
+		(property "Reference" "C5"
 			(at 118.364 64.516 0)
 			(show_name no)
@@
 			(project "PoE_Splitter"
 				(path "/d9db320b-7bcf-482d-be5b-dfde980903b7/135e74f4-e2a5-4ade-99ba-362d75f4aa12"
-					(reference "C14")
+					(reference "C5")
 					(unit 1)
 				)
@@
 		(in_pos_files yes)
 		(dnp no)
-		(property "Reference" "C28"
+		(property "Reference" "C10"
 			(at 125.984 106.426 0)
 			(show_name no)
@@
 			(project "PoE_Splitter"
 				(path "/d9db320b-7bcf-482d-be5b-dfde980903b7/135e74f4-e2a5-4ade-99ba-362d75f4aa12"
-					(reference "C28")
+					(reference "C10")
 					(unit 1)
 				)
@@
 		(in_pos_files yes)
 		(dnp no)
-		(property "Reference" "FB2"
+		(property "Reference" "FB1"
 			(at 198.12 112.776 90)
 			(show_name no)
@@
 			(project "PoE_Splitter"
 				(path "/d9db320b-7bcf-482d-be5b-dfde980903b7/135e74f4-e2a5-4ade-99ba-362d75f4aa12"
-					(reference "FB2")
+					(reference "FB1")
 					(unit 1)
 				)
@@
 		(in_pos_files yes)
 		(dnp no)
-		(property "Reference" "C20"
+		(property "Reference" "C30"
 			(at 212.344 85.598 0)
 			(show_name no)
@@
 			(project "PoE_Splitter"
 				(path "/d9db320b-7bcf-482d-be5b-dfde980903b7/135e74f4-e2a5-4ade-99ba-362d75f4aa12"
-					(reference "C20")
+					(reference "C30")
 					(unit 1)
 				)
@@
 		(in_pos_files yes)
 		(dnp no)
-		(property "Reference" "C16"
+		(property "Reference" "C4"
 			(at 125.984 64.516 0)
 			(show_name no)
@@
 			(project "PoE_Splitter"
 				(path "/d9db320b-7bcf-482d-be5b-dfde980903b7/135e74f4-e2a5-4ade-99ba-362d75f4aa12"
-					(reference "C16")
+					(reference "C4")
 					(unit 1)
 				)
@@
 		(in_pos_files yes)
 		(dnp no)
-		(property "Reference" "RV1"
+		(property "Reference" "RV4"
 			(at 96.774 104.394 0)
 			(show_name no)
@@
 			(project "PoE_Splitter"
 				(path "/d9db320b-7bcf-482d-be5b-dfde980903b7/135e74f4-e2a5-4ade-99ba-362d75f4aa12"
-					(reference "RV1")
+					(reference "RV4")
 					(unit 1)
 				)
@@
 		(in_pos_files yes)
 		(dnp no)
-		(property "Reference" "RV4"
+		(property "Reference" "RV1"
 			(at 84.074 104.394 0)
 			(show_name no)
@@
 			(project "PoE_Splitter"
 				(path "/d9db320b-7bcf-482d-be5b-dfde980903b7/135e74f4-e2a5-4ade-99ba-362d75f4aa12"
-					(reference "RV4")
+					(reference "RV1")
 					(unit 1)
 				)
@@
 		(in_pos_files yes)
 		(dnp no)
-		(property "Reference" "C26"
+		(property "Reference" "C11"
 			(at 118.364 106.426 0)
 			(show_name no)
@@
 			(project "PoE_Splitter"
 				(path "/d9db320b-7bcf-482d-be5b-dfde980903b7/135e74f4-e2a5-4ade-99ba-362d75f4aa12"
-					(reference "C26")
+					(reference "C11")
 					(unit 1)
 				)
@@
 		(in_pos_files yes)
 		(dnp no)
-		(property "Reference" "FB1"
+		(property "Reference" "FB2"
 			(at 198.12 56.896 90)
 			(show_name no)
@@
 			(project "PoE_Splitter"
 				(path "/d9db320b-7bcf-482d-be5b-dfde980903b7/135e74f4-e2a5-4ade-99ba-362d75f4aa12"
-					(reference "FB1")
+					(reference "FB2")
 					(unit 1)
 				)
@@
 		(in_pos_files yes)
 		(dnp no)
-		(property "Reference" "RV3"
+		(property "Reference" "RV2"
 			(at 90.424 104.394 0)
 			(show_name no)
@@
 			(project "PoE_Splitter"
 				(path "/d9db320b-7bcf-482d-be5b-dfde980903b7/135e74f4-e2a5-4ade-99ba-362d75f4aa12"
-					(reference "RV3")
+					(reference "RV2")
 					(unit 1)
 				)
@@
 		(in_pos_files yes)
 		(dnp no)
-		(property "Reference" "D3"
+		(property "Reference" "D6"
 			(at 110.49 84.074 90)
 			(show_name no)
@@
 			(project "PoE_Splitter"
 				(path "/d9db320b-7bcf-482d-be5b-dfde980903b7/135e74f4-e2a5-4ade-99ba-362d75f4aa12"
-					(reference "D3")
+					(reference "D6")
 					(unit 1)
 				)
@@
 		(in_pos_files yes)
 		(dnp no)
-		(property "Reference" "C17"
+		(property "Reference" "C2"
 			(at 129.794 64.516 0)
 			(show_name no)
@@
 			(project "PoE_Splitter"
 				(path "/d9db320b-7bcf-482d-be5b-dfde980903b7/135e74f4-e2a5-4ade-99ba-362d75f4aa12"
-					(reference "C17")
+					(reference "C2")
 					(unit 1)
 				)
@@
 		(in_pos_files yes)
 		(dnp no)
-		(property "Reference" "C18"
+		(property "Reference" "C8"
 			(at 134.874 77.216 0)
 			(show_name no)
@@
 			(project "PoE_Splitter"
 				(path "/d9db320b-7bcf-482d-be5b-dfde980903b7/135e74f4-e2a5-4ade-99ba-362d75f4aa12"
-					(reference "C18")
+					(reference "C8")
 					(unit 1)
 				)
@@
 		(in_pos_files yes)
 		(dnp no)
-		(property "Reference" "D1"
+		(property "Reference" "D5"
 			(at 110.49 101.6 90)
 			(show_name no)
@@
 			(project "PoE_Splitter"
 				(path "/d9db320b-7bcf-482d-be5b-dfde980903b7/135e74f4-e2a5-4ade-99ba-362d75f4aa12"
-					(reference "D1")
+					(reference "D5")
 					(unit 1)
 				)
@@
 		(in_pos_files yes)
 		(dnp no)
-		(property "Reference" "C19"
+		(property "Reference" "C31"
 			(at 184.404 85.598 0)
 			(show_name no)
@@
 			(project "PoE_Splitter"
 				(path "/d9db320b-7bcf-482d-be5b-dfde980903b7/135e74f4-e2a5-4ade-99ba-362d75f4aa12"
-					(reference "C19")
+					(reference "C31")
 					(unit 1)
 				)
@@
 		(in_pos_files yes)
 		(dnp no)
-		(property "Reference" "C27"
+		(property "Reference" "C13"
 			(at 122.174 106.426 0)
 			(show_name no)
@@
 			(project "PoE_Splitter"
 				(path "/d9db320b-7bcf-482d-be5b-dfde980903b7/135e74f4-e2a5-4ade-99ba-362d75f4aa12"
-					(reference "C27")
+					(reference "C13")
 					(unit 1)
 				)
@@
 		(in_pos_files yes)
 		(dnp no)
-		(property "Reference" "C29"
+		(property "Reference" "C12"
 			(at 129.794 106.426 0)
 			(show_name no)
@@
 			(project "PoE_Splitter"
 				(path "/d9db320b-7bcf-482d-be5b-dfde980903b7/135e74f4-e2a5-4ade-99ba-362d75f4aa12"
-					(reference "C29")
+					(reference "C12")
 					(unit 1)
 				)
@@
 		(in_pos_files yes)
 		(dnp no)
-		(property "Reference" "C25"
+		(property "Reference" "C9"
 			(at 134.874 94.996 0)
 			(show_name no)
@@
 			(project "PoE_Splitter"
 				(path "/d9db320b-7bcf-482d-be5b-dfde980903b7/135e74f4-e2a5-4ade-99ba-362d75f4aa12"
-					(reference "C25")
+					(reference "C9")
 					(unit 1)
 				)
@@
 		(in_pos_files yes)
 		(dnp no)
-		(property "Reference" "U2"
+		(property "Reference" "U4"
 			(at 154.432 73.914 0)
 			(show_name no)
@@
 			(project "PoE_Splitter"
 				(path "/d9db320b-7bcf-482d-be5b-dfde980903b7/135e74f4-e2a5-4ade-99ba-362d75f4aa12"
-					(reference "U2")
+					(reference "U4")
 					(unit 1)
 				)
@@
 		(in_pos_files yes)
 		(dnp no)
-		(property "Reference" "RV2"
+		(property "Reference" "RV3"
 			(at 103.124 104.394 0)
 			(show_name no)
@@
 			(project "PoE_Splitter"
 				(path "/d9db320b-7bcf-482d-be5b-dfde980903b7/135e74f4-e2a5-4ade-99ba-362d75f4aa12"
-					(reference "RV2")
-					(unit 1)
-				)
+					(reference "RV3")
+					(unit 1)
+				)

Commit message: add ci
Connections:
- net PRE_VDD renamed VRECT+
- net PRE_VSS renamed VRECT-
Changed lines of the file:
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@@
+	)
+	(symbol
+		(lib_id "PoE_Splitter:VRECT-")
+		(at 177.8 116.84 180)
+		(unit 1)
+		(body_style 1)
+		(exclude_from_sim no)
+		(in_bom yes)
+		(on_board yes)
+		(in_pos_files yes)
+		(dnp no)
+		(property "Reference" "#PWR024"
+			(at 177.8 113.03 0)
+			(hide yes)
+			(show_name no)
+			(do_not_autoplace no)
+			(effects
+				(font
+					(size 1.016 1.016)
+				)
+			)
+		)
+		(property "Value" "VRECT-"
+			(at 177.8 120.65 0)
+			(show_name no)
+			(do_not_autoplace no)
+			(effects
+				(font
+					(size 1.016 1.016)
+				)
+			)
+		)
+		(property "Footprint" ""
+			(at 177.8 116.84 0)
+			(hide yes)
+			(show_name no)
+			(do_not_autoplace no)
+			(effects
+				(font
+					(size 1.27 1.27)
+				)
+			)
+		)
+		(property "Datasheet" ""
+			(at 177.8 116.84 0)
+			(hide yes)
+			(show_name no)
+			(do_not_autoplace no)
+			(effects
+				(font
+					(size 1.27 1.27)
+				)
+			)
+		)
+		(property "Description" "Power symbol creates a global label with name \"VRECT-\""
+			(at 177.8 116.84 0)
+			(hide yes)
+			(show_name no)
+			(do_not_autoplace no)
+			(effects
+				(font
+					(size 1.27 1.27)
+				)
+			)
+		)
+		(pin "1"
+		)
+		(instances
+			(project "PoE_Splitter"
+				(path "/d9db320b-7bcf-482d-be5b-dfde980903b7/135e74f4-e2a5-4ade-99ba-362d75f4aa12"
+					(reference "#PWR024")
+					(unit 1)
+				)
+			)
+		)
 	)
 	(symbol
@@
 	)
 	(symbol
+		(lib_id "PoE_Splitter:VRECT+")
+		(at 177.8 58.42 0)
+		(unit 1)
+		(body_style 1)
+		(exclude_from_sim no)
+		(in_bom yes)
+		(on_board yes)
+		(in_pos_files yes)
+		(dnp no)
+		(property "Reference" "#PWR05"
+			(at 177.8 62.23 0)
+			(hide yes)
+			(show_name no)
+			(do_not_autoplace no)
+			(effects
+				(font
+					(size 1.016 1.016)
+				)
+			)
+		)
+		(property "Value" "VRECT+"
+			(at 177.8 54.864 0)
+			(show_name no)
+			(do_not_autoplace no)
+			(effects
+				(font
+					(size 1.016 1.016)
+				)
+			)
+		)
+		(property "Footprint" ""
+			(at 177.8 58.42 0)
+			(hide yes)
+			(show_name no)
+			(do_not_autoplace no)
+			(effects
+				(font
+					(size 1.27 1.27)
+				)
+			)
+		)
+		(property "Datasheet" ""
+			(at 177.8 58.42 0)
+			(hide yes)
+			(show_name no)
+			(do_not_autoplace no)
+			(effects
+				(font
+					(size 1.27 1.27)
+				)
+			)
+		)
+		(property "Description" "Power symbol creates a global label with name \"VRECT+\""
+			(at 177.8 58.42 0)
+			(hide yes)
+			(show_name no)
+			(do_not_autoplace no)
+			(effects
+				(font
+					(size 1.27 1.27)
+				)
+			)
+		)
+		(pin "1"
+		)
+		(instances
+			(project "PoE_Splitter"
+				(path "/d9db320b-7bcf-482d-be5b-dfde980903b7/135e74f4-e2a5-4ade-99ba-362d75f4aa12"
+					(reference "#PWR05")
+					(unit 1)
+				)
+			)
+		)
+	)
+	(symbol
 		(lib_id "Device:Varistor")
 		(at 96.52 107.95 0)
@@
 	)
 	(symbol
-		(lib_id "PoE_Splitter:PRE_VSS")
-		(at 177.8 116.84 180)
-		(unit 1)
-		(body_style 1)
-		(exclude_from_sim no)
-		(in_bom yes)
-		(on_board yes)
-		(in_pos_files yes)
-		(dnp no)
-		(property "Reference" "#PWR024"
-			(at 177.8 113.03 0)
-			(hide yes)
-			(show_name no)
-			(do_not_autoplace no)
-			(effects
-				(font
-					(size 1.27 1.27)
-				)
-			)
-		)
-		(property "Value" "PRE_VSS"
-			(at 177.8 120.396 0)
-			(show_name no)
-			(do_not_autoplace no)
-			(effects
-				(font
-					(size 1.016 1.016)
-				)
-			)
-		)
-		(property "Footprint" ""
-			(at 177.8 116.84 0)
-			(hide yes)
-			(show_name no)
-			(do_not_autoplace no)
-			(effects
-				(font
-					(size 1.27 1.27)
-				)
-			)
-		)
-		(property "Datasheet" ""
-			(at 177.8 116.84 0)
-			(hide yes)
-			(show_name no)
-			(do_not_autoplace no)
-			(effects
-				(font
-					(size 1.27 1.27)
-				)
-			)
-		)
-		(property "Description" "Power symbol creates a global label with name \"PRE_VSS\""
-			(at 177.8 116.84 0)
-			(hide yes)
-			(show_name no)
-			(do_not_autoplace no)
-			(effects
-				(font
-					(size 1.27 1.27)
-				)
-			)
-		)
-		(pin "1"
-		)
-		(instances
-			(project "PoE_Splitter"
-				(path "/d9db320b-7bcf-482d-be5b-dfde980903b7/135e74f4-e2a5-4ade-99ba-362d75f4aa12"
-					(reference "#PWR024")
-					(unit 1)
-				)
-			)
-		)
-	)
-	(symbol
 		(lib_id "Device:Varistor")
 		(at 90.17 107.95 0)
@@
 					(unit 1)
 				)
-			)
-		)
-	)
-	(symbol
-		(lib_id "PoE_Splitter:PRE_VDD")
-		(at 177.8 58.42 0)
-		(unit 1)
-		(body_style 1)
-		(exclude_from_sim no)
-		(in_bom yes)
-		(on_board yes)
-		(in_pos_files yes)
-		(dnp no)
-		(property "Reference" "#PWR023"
-			(at 177.8 62.23 0)
-			(hide yes)
-			(show_name no)
-			(do_not_autoplace no)
-			(effects
-				(font
-					(size 1.27 1.27)
-				)
-			)
-		)
-		(property "Value" "PRE_VDD"
-			(at 177.8 54.864 0)
-			(show_name no)
-			(do_not_autoplace no)
-			(effects
-				(font
-					(size 1.016 1.016)
-				)
-			)
-		)
-		(property "Footprint" ""
-			(at 177.8 58.42 0)
-			(hide yes)
-			(show_name no)
-			(do_not_autoplace no)
-			(effects
-				(font
-					(size 1.27 1.27)
-				)
-			)
-		)
-		(property "Datasheet" ""
-			(at 177.8 58.42 0)
-			(hide yes)
-			(show_name no)
-			(do_not_autoplace no)
-			(effects
-				(font
-					(size 1.27 1.27)
-				)
-			)
-		)
-		(property "Description" "Power symbol creates a global label with name \"PRE_VDD\""
-			(at 177.8 58.42 0)
-			(hide yes)
-			(show_name no)
-			(do_not_autoplace no)
-			(effects
-				(font
-					(size 1.27 1.27)
-				)
-			)
-		)
-		(pin "1"
-		)
-		(instances
-			(project "PoE_Splitter"
-				(path "/d9db320b-7bcf-482d-be5b-dfde980903b7/135e74f4-e2a5-4ade-99ba-362d75f4aa12"
-					(reference "#PWR023")
-					(unit 1)
-				)

Commit message: add sheet titles
Other:
- company: (none) -> Acha
- title: (none) -> PoE_Splitter
Changed lines of the file:
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@@
 	(generator_version "10.0")
 	(paper "A4")
+	(title_block
+		(title "PoE_Splitter")
+		(date "${CURRENT_DATE}")
+		(rev "${SHORT_SHA}")
+		(company "Acha")
+		(comment 1 "https://github.com/acha666/PoE_Splitter@${BRANCH}")
+		(comment 2 "GPL-3.0 Licensed")
+	)
 	(junction
 		(at 177.8 115.57)
