File: Rectifier.kicad_sch (KiCad schematic)
At the start: 22 parts, among them U4 PD70224

Commit message: fix: pd70224 input connection
Parts:
- added R35: 0Ω, Resistor_SMD:R_1206_3216Metric, symbol Device:R
- U4: symbol Power_Management:PD70224 -> PoE_Splitter:PD70224
Connections:
- net PD+: now also C12.1, C2.2, U4.15 (IN1A), U4.16 (IN1A), U4.27 (IN1A), U4.28 (IN1A); no longer C13.1, C3.2, U4.11 (IN2A), U4.12 (IN2A), U4.31 (IN2A), U4.32 (IN2A)
- net PD-: now also C13.1, C3.2, U4.11 (IN2A), U4.12 (IN2A), U4.31 (IN2A), U4.32 (IN2A); no longer C11.1, C5.2, U4.4 (IN2B), U4.5 (IN2B), U4.6 (IN2B), U4.7 (IN2B)
- net PS+: now also C11.1, C5.2, U4.4 (IN2B), U4.5 (IN2B), U4.6 (IN2B), U4.7 (IN2B); no longer C10.1, C4.2, U4.20 (IN1B), U4.21 (IN1B), U4.22 (IN1B), U4.23 (IN1B)
- net PS-: now also C10.1, C4.2, U4.20 (IN1B), U4.21 (IN1B), U4.22 (IN1B), U4.23 (IN1B); no longer C12.1, C2.2, U4.15 (IN1A), U4.16 (IN1A), U4.27 (IN1A), U4.28 (IN1A)
- net VRECT-: now also R35.2; no longer U4.29 (WA_EN)
- new net: R35.1, U4.29 (WA_EN)
Other:
- moved on the sheet: C3, C4, C8, C9, D5, D6
