File: Brick_Converter.kicad_sch (KiCad schematic)
At the start: 10 parts, among them Q1 BSS127S, U1 VCF4812EBO-120WR3-N

Commit message: 1
Parts:
- added C17: 150uF, Capacitor_THT:CP_Radial_D10.0mm_P5.00mm, symbol Device:C_Polarized
- added C53: 2.2uF, Capacitor_SMD:C_1812_4532Metric, symbol Device:C
- renumbered C3 to C18, C1 to C32, C10 to C37, C4 to C40, R1 to R12, R4 to R16, R2 to R19, R3 to R20
Connections:
- net VOUT+: now also C17.1, C53.1
- net VOUT-: now also C17.2, C53.2
Other:
- moved on the sheet: C40

Commit message: add ci
Changed lines of the file:
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@@
-	)
-	(junction
-		(at 170.18 116.84)
-		(diameter 0)
-		(color 0 0 0 0)
 	)
 	(junction
@@
 	)
 	(junction
-		(at 170.18 78.74)
-		(diameter 0)
-		(color 0 0 0 0)
-	)
-	(junction
 		(at 135.89 88.9)
 		(diameter 0)
@@
 	(wire
 		(pts
-			(xy 170.18 116.84) (xy 182.88 116.84)
-		)
-		(stroke
-			(width 0)
-			(type default)
-		)
-	)
-	(wire
-		(pts
 			(xy 138.43 90.17) (xy 138.43 88.9)
 		)
@@
 		(pts
 			(xy 135.89 106.68) (xy 138.43 106.68)
-		)
-		(stroke
-			(width 0)
-			(type default)
-		)
-	)
-	(wire
-		(pts
-			(xy 170.18 78.74) (xy 182.88 78.74)
 		)
 		(stroke
@@
 			(effects
 				(font
-					(size 1.27 1.27)
+					(size 1.016 1.016)
 				)
 			)
@@
 			(effects
 				(font
-					(size 1.27 1.27)
-				)
-			)
+					(size 1.016 1.016)
+				)
+			)

Commit message: add sheet titles
Other:
- company: (none) -> Acha
- title: (none) -> PoE_Splitter
Changed lines of the file:
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@@
 	(generator_version "10.0")
 	(paper "A4")
+	(title_block
+		(title "PoE_Splitter")
+		(date "${CURRENT_DATE}")
+		(rev "${SHORT_SHA}")
+		(company "Acha")
+		(comment 1 "https://github.com/acha666/PoE_Splitter@${BRANCH}")
+		(comment 2 "GPL-3.0 Licensed")
+	)
 	(junction
 		(at 138.43 116.84)

Commit message: MPQ boost cap value MPQ PG pull-up res all res value unit naming
Parts:
- R12: value 220K -> 220kΩ
- R16: value 33K -> 33kΩ
Changed lines of the file:
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@@
 			)
 		)
-		(property "Value" "220K"
+		(property "Value" "220kΩ"
 			(at 92.202 92.456 0)
 			(show_name no)
@@
 			)
 		)
-		(property "Value" "33K"
+		(property "Value" "33kΩ"
 			(at 92.202 105.156 0)
 			(show_name no)
