File: Brick_Converter.kicad_sch (KiCad schematic)
At the start: 12 parts, among them Q1 BSS127S, U1 VCF4812EBO-120WR3-N

Commit message: minor cap footprint and value changes
Parts:
- C40: value 2.2uF -> 1uF
- C53: value 2.2uF -> 100nF
Changed lines of the file:
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@@
 			)
 		)
-		(property "Value" "2.2uF"
+		(property "Value" "100nF"
 			(at 170.688 100.33 0)
 			(show_name no)
@@
 			)
 		)
-		(property "Value" "2.2uF"
+		(property "Value" "1uF"
 			(at 163.068 100.33 0)
 			(show_name no)
