File: DCDC.kicad_sch (KiCad schematic)
At the start: 24 parts, among them U4 MPQ8875A

Commit message: 1
Parts:
- added C29: 150uF, Capacitor_SMD:CP_Elec_6.3x5.7, symbol Device:C_Polarized
- C26: renamed from C40; value 10uF -> 2.2uF
- C27: renamed from C41; value 10uF -> 2.2uF
- L2: footprint Inductor_SMD:L_Coilcraft_XAL8080-XXX -> Inductor_SMD:L_Chilisin_BWVS00808040
- renumbered C33 to C14, C43 to C15, C44 to C16, C45 to C19, C39 to C20, C34 to C21, C36 to C22, C35 to C23, C46 to C24, C42 to C25, C37 to C42, C48 to C44, C38 to C45, C49 to C50, C47 to C51, R30 to R28, R29 to R30, R28 to R6, R26 to R7, R27 to R8, U4 to U3
Connections:
- net PGND1: now also C29.2
- net PVOUT: now also C29.1
- net Net-(C42-Pad2): now reaches C42.2, R28.2
Other:
- moved on the sheet: C14, C15, C16, C19, C20, C21, C22, C23, C24, C25, C26, C27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

Commit message: add ci
Parts:
- added R31, R32: 10kΩ, Resistor_SMD:R_0603_1608Metric, symbol Device:R_Small
- added R33, R34: 22Ω, Resistor_SMD:R_0603_1608Metric, symbol Device:R_Small
- added U5: USBLC6-2P6, Package_TO_SOT_SMD:SOT-666, symbol Power_Protection:USBLC6-2P6
Connections:
- net MPS_VCC: now also R31.1, R32.1, U5.5 (VBUS)
- net PGND1: now also U5.2 (GND)
- net SCL: now also U5.6 (I/O1); no longer U3.12 (SCL)
- net SDA: now also U5.4 (I/O2); no longer U3.11 (SDA)
- net Net-(C42-Pad2): no longer names the net of C42.2, R28.2
- net PVOUT renamed AUX_OUT+
- new net: R34.2, U5.3 (I/O2)
- new net: R33.2, U5.1 (I/O1)
- new net MPS_SCL: R32.2, R33.1, U3.12 (SCL)
- new net MPS_SDA: R31.2, R34.1, U3.11 (SDA)

Commit message: add sheet titles
Other:
- company: (none) -> Acha
- title: (none) -> PoE_Splitter
Changed lines of the file:
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@@
 	(generator_version "10.0")
 	(paper "A4")
+	(title_block
+		(title "PoE_Splitter")
+		(date "${CURRENT_DATE}")
+		(rev "${SHORT_SHA}")
+		(company "Acha")
+		(comment 1 "https://github.com/acha666/PoE_Splitter@${BRANCH}")
+		(comment 2 "GPL-3.0 Licensed")
+	)
 	(junction
 		(at 72.39 76.2)

Commit message: MPQ boost cap value MPQ PG pull-up res all res value unit naming
Parts:
- C21, C23: value 10nF -> 100nF
- R30: value 110kΩ -> 10kΩ; now not fitted
- R31, R32: value 10kΩ -> 5.1kΩ
Changed lines of the file:
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@@
 			)
 		)
-		(property "Value" "10nF"
+		(property "Value" "100nF"
 			(at 124.714 58.928 0)
 			(show_name no)
@@
 			)
 		)
-		(property "Value" "10kΩ"
+		(property "Value" "5.1kΩ"
 			(at 154.432 124.206 0)
 			(show_name no)
@@
 			)
 		)
-		(property "Value" "10nF"
+		(property "Value" "100nF"
 			(at 147.574 58.928 0)
 			(show_name no)
@@
 			)
 		)
-		(property "Value" "10kΩ"
+		(property "Value" "5.1kΩ"
 			(at 148.082 124.206 0)
 			(show_name no)
@@
 		(on_board yes)
 		(in_pos_files yes)
-		(dnp no)
+		(dnp yes)
 		(property "Reference" "R30"
 			(at 174.752 90.424 0)
@@
 			)
 		)
-		(property "Value" "110kΩ"
+		(property "Value" "10kΩ"
 			(at 174.752 92.456 0)
 			(show_name no)
