File: DCDC.kicad_sch (KiCad schematic)
At the start: 30 parts, among them U3 MPQ8875A, U5 USBLC6-2P6

Commit message: change C29 footprint XT30 3d model position
Parts:
- C29: footprint Capacitor_SMD:CP_Elec_6.3x5.7 -> Capacitor_SMD:CP_Elec_6.3x7.7
Changed lines of the file:
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@@
 			)
 		)
-		(property "Footprint" "Capacitor_SMD:CP_Elec_6.3x5.7"
+		(property "Footprint" "Capacitor_SMD:CP_Elec_6.3x7.7"
 			(at 246.0752 92.71 0)
 			(hide yes)
