File: PD_Frontend.kicad_sch (KiCad schematic)
At the start: 17 parts, among them U3 TPS2372

Commit message: 1
Parts:
- C6: renamed from C21; KiLib_Generator (none) -> capacitor/THT/other
- renumbered C13 to C1, C24 to C33, C22 to C34, C23 to C35, C32 to C7, D4 to D7, R13 to R1, R20 to R10, R19 to R11, R22 to R13, R21 to R14, R15 to R17, R18 to R2, R17 to R9, U3 to U2
Changed lines of the file:
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@@
 		(in_pos_files yes)
 		(dnp no)
-		(property "Reference" "C32"
+		(property "Reference" "C7"
 			(at 185.928 85.598 0)
 			(show_name no)
@@
 			(project "PoE_Splitter"
 				(path "/d9db320b-7bcf-482d-be5b-dfde980903b7/b97941c7-46c2-4c9c-aec0-f8a528a236ea"
-					(reference "C32")
+					(reference "C7")
 					(unit 1)
 				)
@@
 		(in_pos_files yes)
 		(dnp no)
-		(property "Reference" "R22"
+		(property "Reference" "R13"
 			(at 118.872 109.474 0)
 			(show_name no)
@@
 			(project "PoE_Splitter"
 				(path "/d9db320b-7bcf-482d-be5b-dfde980903b7/b97941c7-46c2-4c9c-aec0-f8a528a236ea"
-					(reference "R22")
+					(reference "R13")
 					(unit 1)
 				)
@@
 		(in_pos_files yes)
 		(dnp no)
-		(property "Reference" "R17"
+		(property "Reference" "R9"
 			(at 87.122 103.124 0)
 			(show_name no)
@@
 			(project "PoE_Splitter"
 				(path "/d9db320b-7bcf-482d-be5b-dfde980903b7/b97941c7-46c2-4c9c-aec0-f8a528a236ea"
-					(reference "R17")
+					(reference "R9")
 					(unit 1)
 				)
@@
 		(in_pos_files yes)
 		(dnp no)
-		(property "Reference" "R20"
+		(property "Reference" "R10"
 			(at 93.472 109.474 0)
 			(show_name no)
@@
 			(project "PoE_Splitter"
 				(path "/d9db320b-7bcf-482d-be5b-dfde980903b7/b97941c7-46c2-4c9c-aec0-f8a528a236ea"
-					(reference "R20")
+					(reference "R10")
 					(unit 1)
 				)
@@
 		(in_pos_files yes)
 		(dnp no)
-		(property "Reference" "C22"
+		(property "Reference" "C34"
 			(at 200.914 85.598 0)
 			(show_name no)
@@
 			(project "PoE_Splitter"
 				(path "/d9db320b-7bcf-482d-be5b-dfde980903b7/b97941c7-46c2-4c9c-aec0-f8a528a236ea"
-					(reference "C22")
+					(reference "C34")
 					(unit 1)
 				)
@@
 		(in_pos_files yes)
 		(dnp no)
-		(property "Reference" "U3"
+		(property "Reference" "U2"
 			(at 128.016 65.278 0)
 			(show_name no)
@@
 			(project "PoE_Splitter"
 				(path "/d9db320b-7bcf-482d-be5b-dfde980903b7/b97941c7-46c2-4c9c-aec0-f8a528a236ea"
-					(reference "U3")
+					(reference "U2")
 					(unit 1)
 				)
@@
 		(in_pos_files yes)
 		(dnp no)
-		(property "Reference" "C23"
+		(property "Reference" "C35"
 			(at 208.534 85.598 0)
 			(show_name no)
@@
 			(project "PoE_Splitter"
 				(path "/d9db320b-7bcf-482d-be5b-dfde980903b7/b97941c7-46c2-4c9c-aec0-f8a528a236ea"
-					(reference "C23")
+					(reference "C35")
 					(unit 1)
 				)
@@
 		(in_pos_files yes)
 		(dnp no)
-		(property "Reference" "C21"
+		(property "Reference" "C6"
 			(at 193.548 85.598 0)
 			(show_name no)
@@
 			)
 		)
+		(property "KiLib_Generator" "capacitor/THT/other"
+			(at 193.04 87.63 0)
+			(hide yes)
+			(show_name no)
+			(do_not_autoplace no)
+			(effects
+				(font
+					(size 1.27 1.27)
+				)
+			)
+		)
 		(pin "2"
 		)
@@
 			(project "PoE_Splitter"
 				(path "/d9db320b-7bcf-482d-be5b-dfde980903b7/b97941c7-46c2-4c9c-aec0-f8a528a236ea"
-					(reference "C21")
+					(reference "C6")
 					(unit 1)
 				)
@@
 		(in_pos_files yes)
 		(dnp no)
-		(property "Reference" "R21"
+		(property "Reference" "R14"
 			(at 106.68 108.458 0)
 			(show_name no)
@@
 			(project "PoE_Splitter"
 				(path "/d9db320b-7bcf-482d-be5b-dfde980903b7/b97941c7-46c2-4c9c-aec0-f8a528a236ea"
-					(reference "R21")
+					(reference "R14")
 					(unit 1)
 				)
@@
 		(in_pos_files yes)
 		(dnp yes)
-		(property "Reference" "R15"
+		(property "Reference" "R17"
 			(at 164.592 89.154 0)
 			(show_name no)
@@
 			(project "PoE_Splitter"
 				(path "/d9db320b-7bcf-482d-be5b-dfde980903b7/b97941c7-46c2-4c9c-aec0-f8a528a236ea"
-					(reference "R15")
+					(reference "R17")
 					(unit 1)
 				)
@@
 		(in_pos_files yes)
 		(dnp no)
-		(property "Reference" "R13"
+		(property "Reference" "R1"
 			(at 93.472 65.024 0)
 			(show_name no)
@@
 			(project "PoE_Splitter"
 				(path "/d9db320b-7bcf-482d-be5b-dfde980903b7/b97941c7-46c2-4c9c-aec0-f8a528a236ea"
-					(reference "R13")
+					(reference "R1")
 					(unit 1)
 				)
@@
 		(in_pos_files yes)
 		(dnp no)
-		(property "Reference" "C24"
+		(property "Reference" "C33"
 			(at 216.154 85.598 0)
 			(show_name no)
@@
 			(project "PoE_Splitter"
 				(path "/d9db320b-7bcf-482d-be5b-dfde980903b7/b97941c7-46c2-4c9c-aec0-f8a528a236ea"
-					(reference "C24")
+					(reference "C33")
 					(unit 1)
 				)
@@
 		(in_pos_files yes)
 		(dnp no)
-		(property "Reference" "R19"
+		(property "Reference" "R11"
 			(at 112.522 103.124 0)
 			(show_name no)
@@
 			(project "PoE_Splitter"
 				(path "/d9db320b-7bcf-482d-be5b-dfde980903b7/b97941c7-46c2-4c9c-aec0-f8a528a236ea"
-					(reference "R19")
+					(reference "R11")
 					(unit 1)
 				)
@@
 		(in_pos_files yes)
 		(dnp yes)
-		(property "Reference" "R18"
+		(property "Reference" "R2"
 			(at 99.822 103.124 0)
 			(show_name no)
@@
 			(project "PoE_Splitter"
 				(path "/d9db320b-7bcf-482d-be5b-dfde980903b7/b97941c7-46c2-4c9c-aec0-f8a528a236ea"
-					(reference "R18")
+					(reference "R2")
 					(unit 1)
 				)
@@
 		(in_pos_files yes)
 		(dnp no)
-		(property "Reference" "D4"
+		(property "Reference" "D7"
 			(at 166.37 111.506 0)
 			(show_name no)
@@
 			(project "PoE_Splitter"
 				(path "/d9db320b-7bcf-482d-be5b-dfde980903b7/b97941c7-46c2-4c9c-aec0-f8a528a236ea"
-					(reference "D4")
+					(reference "D7")
 					(unit 1)
 				)
@@
 		(in_pos_files yes)
 		(dnp no)
-		(property "Reference" "C13"
+		(property "Reference" "C1"
 			(at 111.76 63.5 90)
 			(show_name no)
@@
 			(project "PoE_Splitter"
 				(path "/d9db320b-7bcf-482d-be5b-dfde980903b7/b97941c7-46c2-4c9c-aec0-f8a528a236ea"
-					(reference "C13")
-					(unit 1)
-				)
+					(reference "C1")
+					(unit 1)
+				)

Commit message: add ci
Changed lines of the file:
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@@
 			(effects
 				(font
-					(size 1.27 1.27)
+					(size 1.016 1.016)
 				)
 				(justify left)
@@
 			(effects
 				(font
-					(size 1.27 1.27)
+					(size 1.016 1.016)
 				)
 				(justify left)

Commit message: add sheet titles
Other:
- company: (none) -> Acha
- title: (none) -> PoE_Splitter
Changed lines of the file:
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@@
 	(generator_version "10.0")
 	(paper "A4")
+	(title_block
+		(title "PoE_Splitter")
+		(date "${CURRENT_DATE}")
+		(rev "${SHORT_SHA}")
+		(company "Acha")
+		(comment 1 "https://github.com/acha666/PoE_Splitter@${BRANCH}")
+		(comment 2 "GPL-3.0 Licensed")
+	)
 	(junction
 		(at 157.48 86.36)

Commit message: MPQ boost cap value MPQ PG pull-up res all res value unit naming
Parts:
- R1: value 24.9K -> 24.9kΩ
- R10: value 90.9R -> 90.9Ω
- R11: value 49.9K -> 49.9kΩ
- R13, R17, R2: value 0R -> 0Ω
- R14: value 1.3K -> 1.3kΩ
- R9: value 63.4R -> 63.4Ω
Changed lines of the file:
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@@
 			)
 		)
-		(property "Value" "0R"
+		(property "Value" "0Ω"
 			(at 118.872 111.506 0)
 			(show_name no)
@@
 			)
 		)
-		(property "Value" "63.4R"
+		(property "Value" "63.4Ω"
 			(at 87.122 105.156 0)
 			(show_name no)
@@
 			)
 		)
-		(property "Value" "90.9R"
+		(property "Value" "90.9Ω"
 			(at 93.472 111.506 0)
 			(show_name no)
@@
 			)
 		)
-		(property "Value" "1.3K"
+		(property "Value" "1.3kΩ"
 			(at 106.68 110.49 0)
 			(show_name no)
@@
 			)
 		)
-		(property "Value" "0R"
+		(property "Value" "0Ω"
 			(at 164.592 91.186 0)
 			(show_name no)
@@
 			)
 		)
-		(property "Value" "24.9K"
+		(property "Value" "24.9kΩ"
 			(at 93.472 67.056 0)
 			(show_name no)
@@
 			)
 		)
-		(property "Value" "49.9K"
+		(property "Value" "49.9kΩ"
 			(at 112.522 105.156 0)
 			(show_name no)
@@
 			)
 		)
-		(property "Value" "0R"
+		(property "Value" "0Ω"
 			(at 99.822 105.156 0)
 			(show_name no)
