File: PD_Frontend.kicad_sch (KiCad schematic)
At the start: 17 parts, among them U2 TPS2372

Commit message: minor cap footprint and value changes
Parts:
- C34: value 2.2uF -> 1uF
- C35: value 2.2uF -> 100nF
Changed lines of the file:
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@@
 			)
 		)
-		(property "Value" "2.2uF"
+		(property "Value" "1uF"
 			(at 201.168 90.17 0)
 			(show_name no)
@@
 			)
 		)
-		(property "Value" "2.2uF"
+		(property "Value" "100nF"
 			(at 208.788 90.17 0)
 			(show_name no)
